File: v1.0/rng.1.0.brd (EAGLE design)
At the start: 50 x 25 mm, 43 parts, among them IC1 3.3v VREG, IC2 CC2531, IC3 AP3105, X1 32MHz

Commit message: fix typo in part number AP3105->AP3015
Parts:
- IC3: value AP3105 -> AP3015
Changed lines of the file:
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@@
 <attribute name="NAME" x="39.265" y="14.635" size="0.6096" layer="25"/>
 </element>
-<element name="IC3" library="playa" package="SOT23-5" value="AP3105" x="41.6" y="10.7" smashed="yes">
+<element name="IC3" library="playa" package="SOT23-5" value="AP3015" x="41.6" y="10.7" smashed="yes">
 <attribute name="NAME" x="41" y="10.4" size="0.6096" layer="21"/>
 </element>
