File: v1.0/rng.1.0.sch (EAGLE design)
At the start: 43 parts, among them IC1 3.3v VREG, IC2 CC2531, IC3 AP3105, X1 32MHz

Commit message: fix typo in part number AP3105->AP3015
Parts:
- IC3: value AP3105 -> AP3015; device playa:AP3105 -> playa:AP3015
Changed lines of the file:
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@@
 <part name="T2" library="transistor-neu-to92" deviceset="*-NPN-" device="SOT23-BEC" technology="BCF32"/>
 <part name="R11" library="rcl" deviceset="R-US_" device="R0603" value="470k"/>
-<part name="IC3" library="playa" deviceset="AP3105" device=""/>
+<part name="IC3" library="playa" deviceset="AP3015" device=""/>
 <part name="+3V4" library="supply1" deviceset="+3V3" device=""/>
 <part name="SUPPLY21" library="supply2" deviceset="GND" device=""/>
